File: DigiLight.sch (KiCad schematic (older format))
At the start: 69 parts, among them IC1 MAX9814 Module, J1 IN_1, J2 IN_2, J3 POWER (5V/3A), J4 APU-2, J5 112J-TDAR-R-Micro_SD_Card, J6 WS2811, Q1 BC846, Q2 BC846, Q3 BC846, Q4 IRLML6402, Q5 BC846, SW1 Encoder_Switch, SW2 MENU, U1 LM358, U2 LM358, U3 4066, U4 AMS1117-3.3, U5 ATmega32-16AU, U6 TSOP43xx, Y1 16MHz

Commit message: Refactoring input circuit, reassigned MC pins, replace LCD footprint, create PCB template
Parts:
- removed C5: 100.0, Capacitor_THT:CP_Radial_D4.0mm_P1.50mm, symbol Device:CP
- removed Q2: BC846, Package_TO_SOT_SMD:SOT-23, symbol Transistor_BJT:BC846
- removed R10, R11, R12: 15K, Resistor_SMD:R_1206_3216Metric, symbol Device:R
- removed R14: 2.2K, Resistor_SMD:R_1206_3216Metric, symbol Device:R
- removed R16: 240K, Resistor_SMD:R_1206_3216Metric, symbol Device:R
- removed U2: LM358, Package_SO:SOIC-8_3.9x4.9mm_P1.27mm, symbol Amplifier_Operational:LM358
- added C1, C10, C11, C3, C6: 0.1, Capacitor_SMD:C_1206_3216Metric, symbol Device:C
- added C8: 1.0, Capacitor_SMD:C_1206_3216Metric, symbol Device:C
- added C9: 1000.0, Capacitor_THT:CP_Radial_D8.0mm_P5.00mm, symbol Device:CP
- added D1, D2: 1N4448W, Diode_SMD:D_SOD-123, symbol Diode:1N4448W
- added R13: 10K, Resistor_SMD:R_1206_3216Metric, symbol Device:R
- added R7, R8: 15K, Resistor_SMD:R_1206_3216Metric, symbol Device:R
- added unit 2 of U1
- C12: renamed from C4; footprint Capacitor_THT:CP_Radial_D4.0mm_P1.50mm -> Capacitor_SMD:CP_Elec_6.3x5.4
- C2: renamed from C1; value 470.0 -> 1000.0; footprint Capacitor_Tantalum_SMD:CP_EIA-7360-38_Kemet-E_Pad2.25x4.25mm_HandSolder -> Capacitor_THT:CP_Radial_D8.0mm_P5.00mm
- C7: value 2.2 -> 0.1
- LCD1: footprint Display:WC1602A -> ExternalLib:WC1602A_4_data
- R5: renamed from R3; value 1.8K -> 1K
- R6: value 1.8K -> 15K
- renumbered C6 to C13, C8 to C14, C10 to C15, C9 to C16, C11 to C17, C15 to C18, C12 to C19, C13 to C20, C17 to C21, C16 to C22, C14 to C23, C18 to C24, C2 to C4, C3 to C5, Q3 to Q2, Q4 to Q3, Q5 to Q4, R7 to R10, R8 to R11, R13 to R12, R15 to R14, R17 to R15, R18 to R16, R20 to R17, R19 to R18, R21 to R19, R22 to R20, R24 to R21, R23 to R22, R25 to R23, R26 to R24, R4 to R3, R5 to R4, U3 to U1, U1 to U2, U4 to U3, U5 to U4, U6 to U5
Connections:
- net labels added: AGC
- net labels removed: AGC1, AGC2
- no-connect marks 13 -> 14
Other:
- moved on the sheet: C12, C13, C14, C15, C16, C17, C18, C19, C20, C21, C22, C23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

Commit message: Tracing PCB finished
Parts:
- removed D1, D2: 1N4448W, Diode_SMD:D_SOD-123, symbol Diode:1N4448W
- added C11, C16, C8: 0.1, Capacitor_SMD:C_1206_3216Metric, symbol Device:C
- added D1, D2: 1N4148WS, Diode_SMD:D_SOD-323, symbol Diode:1N4148WS
- J3: footprint (none) -> ExternalLib:DC-044
- J6: footprint Connector_JST:JST_XH_B3B-XH-AM_1x03_P2.50mm_Vertical -> Connector_JST:JST_EH_S3B-EH_1x03_P2.50mm_Horizontal
- L1: footprint Inductor_SMD:L_2816_7142Metric -> Inductor_SMD:L_1210_3225Metric
- renumbered C9 to C10, C10 to C13, C11 to C14, C13 to C15, C14 to C17, C15 to C18, C16 to C19, C3 to C2, C17 to C20, C18 to C21, C19 to C22, C20 to C23, C21 to C24, C22 to C25, C23 to C26, C24 to C27, C2 to C3, C7 to C4, C4 to C5, C5 to C6, C6 to C7, C8 to C9
Connections:
- wire segments 250 -> 256
Other:
- moved on the sheet: C1, C13, C14, C2, C4, NT1, U1E

Commit message: Final trace
Parts:
- C27: value 100 -> 4.7uF
Changed lines of the file:
@@
 P 10650 1850
 F 0 "C27" H 10765 1896 50  0000 L CNN
-F 1 "100" H 10765 1805 50  0000 L CNN
+F 1 "4.7uF" H 10765 1805 50  0000 L CNN
 F 2 "Capacitor_SMD:C_1206_3216Metric" H 10688 1700 50  0001 C CNN
 F 3 "~" H 10650 1850 50  0001 C CNN

Commit message: Recalculated 3rd order Sallen-Key Low-pass filter
Parts:
- C18: value 0.015 -> 0.01
- C21: value 6800 -> 5600
- C24: value 100 -> 1000
- R15: value 9.1K -> 4.7K
- R16: value 100K -> 30K
- R17: value 27K -> 10K
Changed lines of the file:
@@
 P 4600 1250
 F 0 "R15" V 4500 1250 50  0000 C CNN
-F 1 "9.1K" V 4700 1250 50  0000 C CNN
+F 1 "4.7K" V 4700 1250 50  0000 C CNN
 F 2 "Resistor_SMD:R_1206_3216Metric" V 4530 1250 50  0001 C CNN
 F 3 "~" H 4600 1250 50  0001 C CNN
@@
 P 5100 1250
 F 0 "R16" V 5000 1250 50  0000 C CNN
-F 1 "100K" V 5200 1250 50  0000 C CNN
+F 1 "30K" V 5200 1250 50  0000 C CNN
 F 2 "Resistor_SMD:R_1206_3216Metric" V 5030 1250 50  0001 C CNN
 F 3 "~" H 5100 1250 50  0001 C CNN
@@
 P 5600 1250
 F 0 "R17" V 5500 1250 50  0000 C CNN
-F 1 "27K" V 5700 1250 50  0000 C CNN
+F 1 "10K" V 5700 1250 50  0000 C CNN
 F 2 "Resistor_SMD:R_1206_3216Metric" V 5530 1250 50  0001 C CNN
 F 3 "~" H 5600 1250 50  0001 C CNN
@@
 P 4850 1650
 F 0 "C18" H 4965 1696 50  0000 L CNN
-F 1 "0.015" H 4965 1605 50  0000 L CNN
+F 1 "0.01" H 4965 1605 50  0000 L CNN
 F 2 "Capacitor_SMD:C_1206_3216Metric" H 4888 1500 50  0001 C CNN
 F 3 "~" H 4850 1650 50  0001 C CNN
@@
 P 5850 1650
 F 0 "C24" H 5965 1696 50  0000 L CNN
-F 1 "100" H 5965 1605 50  0000 L CNN
+F 1 "1000" H 5965 1605 50  0000 L CNN
 F 2 "Capacitor_SMD:C_1206_3216Metric" H 5888 1500 50  0001 C CNN
 F 3 "~" H 5850 1650 50  0001 C CNN
@@
 P 5600 850
 F 0 "C21" V 5450 800 50  0000 L CNN
-F 1 "6800" V 5750 750 50  0000 L CNN
+F 1 "5600" V 5750 750 50  0000 L CNN
 F 2 "Capacitor_SMD:C_1206_3216Metric" H 5638 700 50  0001 C CNN
 F 3 "~" H 5600 850 50  0001 C CNN
@@
 U 1 1 5F23AA5A
 P 3300 900
-F 0 "R13" H 3400 950 50  0000 C CNN
+F 0 "R13" H 3450 950 50  0000 C CNN
 F 1 "10K" H 3450 850 50  0000 C CNN
 F 2 "Resistor_SMD:R_1206_3216Metric" V 3230 900 50  0001 C CNN
@@
 Wire Wire Line
 	1850 1100 1950 1100
-$Comp
-L Device:R R7
-U 1 1 5E8F5BC6
-P 1950 1300
-F 0 "R7" H 2050 1350 50  0000 C CNN
-F 1 "15K" H 2100 1250 50  0000 C CNN
-F 2 "Resistor_SMD:R_1206_3216Metric" V 1880 1300 50  0001 C CNN
-F 3 "~" H 1950 1300 50  0001 C CNN
-	1    1950 1300
-	1    0    0    -1
-$EndComp
 $Comp
 L Device:R R6
@@
 U 1 1 5E790E31
 P 1350 2700
-F 0 "R4" V 1250 2700 50  0000 C CNN
-F 1 "1.8K" V 1450 2700 50  0000 C CNN
+F 0 "R4" V 1450 2700 50  0000 C CNN
+F 1 "1.8K" V 1350 2700 50  0000 C CNN
 F 2 "Resistor_SMD:R_1206_3216Metric" V 1280 2700 50  0001 C CNN
 F 3 "~" H 1350 2700 50  0001 C CNN
@@
 U 1 1 5E6C4444
 P 1350 1300
-F 0 "R2" V 1250 1300 50  0000 C CNN
-F 1 "1.8K" V 1450 1300 50  0000 C CNN
+F 0 "R2" V 1450 1300 50  0000 C CNN
+F 1 "1.8K" V 1350 1300 50  0000 C CNN
 F 2 "Resistor_SMD:R_1206_3216Metric" V 1280 1300 50  0001 C CNN
 F 3 "~" H 1350 1300 50  0001 C CNN
@@
 P 1350 2500
 F 0 "R3" V 1250 2500 50  0000 C CNN
-F 1 "1.8K" V 1450 2500 50  0000 C CNN
+F 1 "1.8K" V 1350 2500 50  0000 C CNN
 F 2 "Resistor_SMD:R_1206_3216Metric" V 1280 2500 50  0001 C CNN
 F 3 "~" H 1350 2500 50  0001 C CNN
@@
 U 1 1 5E59B320
 P 3050 3300
-F 0 "R12" H 3150 3350 50  0000 C CNN
+F 0 "R12" H 3200 3350 50  0000 C CNN
 F 1 "2.2K" H 3200 3250 50  0000 C CNN
 F 2 "Resistor_SMD:R_1206_3216Metric" V 2980 3300 50  0001 C CNN
@@
 P 1350 1100
 F 0 "R1" V 1250 1100 50  0000 C CNN
-F 1 "1.8K" V 1450 1100 50  0000 C CNN
+F 1 "1.8K" V 1350 1100 50  0000 C CNN
 F 2 "Resistor_SMD:R_1206_3216Metric" V 1280 1100 50  0001 C CNN
 F 3 "~" H 1350 1100 50  0001 C CNN
@@
 	1    0    0    -1
 $EndComp
+$Comp
+L Device:R R7
+U 1 1 5E8F5BC6
+P 1950 1300
+F 0 "R7" H 2050 1350 50  0000 C CNN
+F 1 "15K" H 2100 1250 50  0000 C CNN
+F 2 "Resistor_SMD:R_1206_3216Metric" V 1880 1300 50  0001 C CNN
+F 3 "~" H 1950 1300 50  0001 C CNN
+	1    1950 1300
+	1    0    0    -1
+$EndComp

Commit message: Update models, pcb build finish, change output key.
Parts:
- added C28: 2200, Capacitor_SMD:C_1206_3216Metric, symbol Device:C
- J1, J2: symbol PJ-307:AudioJack-PJ-307 -> DigiLight-rescue:AudioJack-PJ-307-PJ-307
- R22: value 1K -> 10K
Connections:
- net GND: no longer R23.1
- net MOSI: now also Q4.2 (E); no longer Q4.3 (C)
- net VPP: now also R23.2
- net WS_LOCK: now also R22.2, C28.2; no longer R22.1
- net at Q4.1 (B): now also R22.1, C28.1; no longer R22.2
- new net: J6.2 (Pin_2), Q4.3 (C), R23.1
Other:
- moved on the sheet: J6, Q4, R22, R23
Changed lines of the file:
@@
 	8600 5700 9250 5700
-$Comp
-L power:VPP #PWR058
-U 1 1 5ED3C80C
-P 10100 2650
-F 0 "#PWR058" H 10100 2500 50  0001 C CNN
-F 1 "VPP" V 10100 2850 50  0000 C CNN
-F 2 "" H 10100 2650 50  0001 C CNN
-F 3 "" H 10100 2650 50  0001 C CNN
-	1    10100 2650
-	0    -1   -1   0
-$EndComp
 $Comp
 L power:GND #PWR059
 U 1 1 5ED41E3D
-P 10100 3150
-F 0 "#PWR059" H 10100 2900 50  0001 C CNN
-F 1 "GND" H 10100 3000 50  0000 C CNN
-F 2 "" H 10100 3150 50  0001 C CNN
-F 3 "" H 10100 3150 50  0001 C CNN
-	1    10100 3150
+P 10450 3200
+F 0 "#PWR059" H 10450 2950 50  0001 C CNN
+F 1 "GND" H 10450 3050 50  0000 C CNN
+F 2 "" H 10450 3200 50  0001 C CNN
+F 3 "" H 10450 3200 50  0001 C CNN
+	1    10450 3200
 	1    0    0    -1
 $EndComp
@@
 L Transistor_BJT:BC846 Q4
 U 1 1 5EDDD9B8
-P 9350 2850
-F 0 "Q4" V 9550 2900 50  0000 L CNN
-F 1 "BC846" V 9550 2550 50  0000 L CNN
-F 2 "Package_TO_SOT_SMD:SOT-23" H 9550 2775 50  0001 L CIN
-F 3 "https://assets.nexperia.com/documents/data-sheet/BC846_SER.pdf" H 9350 2850 50  0001 L CNN
-	1    9350 2850
-	0    -1   -1   0
+P 9550 3150
+F 0 "Q4" V 9450 3000 50  0000 L CNN
+F 1 "BC846" V 9750 3200 50  0000 L CNN
+F 2 "Package_TO_SOT_SMD:SOT-23" H 9750 3075 50  0001 L CIN
+F 3 "https://assets.nexperia.com/documents/data-sheet/BC846_SER.pdf" H 9550 3150 50  0001 L CNN
+	1    9550 3150
+	0    1    1    0
 $EndComp
 $Comp
 L Device:R R23
 U 1 1 5EDE25DA
-P 9750 3000
-F 0 "R23" H 9650 2950 50  0000 C CNN
-F 1 "1K" H 9650 3050 50  0000 C CNN
-F 2 "Resistor_SMD:R_1206_3216Metric" V 9680 3000 50  0001 C CNN
-F 3 "~" H 9750 3000 50  0001 C CNN
-	1    9750 3000
+P 9850 2850
+F 0 "R23" H 9700 2800 50  0000 C CNN
+F 1 "1K" H 9700 2900 50  0000 C CNN
+F 2 "Resistor_SMD:R_1206_3216Metric" V 9780 2850 50  0001 C CNN
+F 3 "~" H 9850 2850 50  0001 C CNN
+	1    9850 2850
 	-1   0    0    1
 $EndComp
-$Comp
-L power:GND #PWR054
-U 1 1 5EE156A2
-P 9750 3150
-F 0 "#PWR054" H 9750 2900 50  0001 C CNN
-F 1 "GND" H 9750 3000 50  0000 C CNN
-F 2 "" H 9750 3150 50  0001 C CNN
-F 3 "" H 9750 3150 50  0001 C CNN
-	1    9750 3150
-	1    0    0    -1
-$EndComp
-Wire Wire Line
-	9550 2750 9750 2750
-Wire Wire Line
-	9750 2850 9750 2750
-Connection ~ 9750 2750
-Wire Wire Line
-	9750 2750 10100 2750
-Wire Wire Line
-	10100 3150 10100 2850
+Wire Wire Line
+	10450 3200 10450 2900
 $Comp
 L Device:R R22
 U 1 1 5EE4155A
-P 9100 3050
-F 0 "R22" V 9200 3050 50  0000 C CNN
-F 1 "1K" V 9000 3050 50  0000 C CNN
-F 2 "Resistor_SMD:R_1206_3216Metric" V 9030 3050 50  0001 C CNN
-F 3 "~" H 9100 3050 50  0001 C CNN
-	1    9100 3050
-	0    -1   -1   0
-$EndComp
-Wire Wire Line
-	9250 3050 9350 3050
-Wire Wire Line
-	8600 2750 9150 2750
-Wire Wire Line
-	8950 3050 8600 3050
+P 9150 2950
+F 0 "R22" V 9050 2950 50  0000 C CNN
+F 1 "10K" V 9250 2950 50  0000 C CNN
+F 2 "Resistor_SMD:R_1206_3216Metric" V 9080 2950 50  0001 C CNN
+F 3 "~" H 9150 2950 50  0001 C CNN
+	1    9150 2950
+	0    1    1    0
+$EndComp
 NoConn ~ 9000 3800
 NoConn ~ 9000 4500
@@
 $EndComp
 Connection ~ 9750 4950
-Text Label 8600 2750 0    50   ~ 0
+Text Label 8500 3250 0    50   ~ 0
 MOSI
-Text Label 8600 3050 0    50   ~ 0
+Text Label 8500 2750 0    50   ~ 0
 WS_LOCK
 Wire Wire Line
@@
 	1050 2900 1100 2900
 $Comp
-L PJ-307:AudioJack-PJ-307 J2
+L DigiLight-rescue:AudioJack-PJ-307-PJ-307 J2
 U 1 1 5E7AB5AA
 P 650 2450
@@
 	1050 1100 1200 1100
 $Comp
-L PJ-307:AudioJack-PJ-307 J1
+L DigiLight-rescue:AudioJack-PJ-307-PJ-307 J1
 U 1 1 5E749281
 P 650 1050
@@
 L Connector_Generic:Conn_01x03 J6
 U 1 1 5ED20E74
-P 10300 2750
-F 0 "J6" H 10250 2950 50  0000 L CNN
-F 1 "WS2811" V 10400 2600 50  0000 L CNN
-F 2 "Connector_JST:JST_EH_S3B-EH_1x03_P2.50mm_Horizontal" H 10300 2750 50  0001 C CNN
-F 3 "~" H 10300 2750 50  0001 C CNN
-	1    10300 2750
+P 10650 2800
+F 0 "J6" H 10600 3000 50  0000 L CNN
+F 1 "WS2811" V 10750 2650 50  0000 L CNN
+F 2 "Connector_JST:JST_EH_S3B-EH_1x03_P2.50mm_Horizontal" H 10650 2800 50  0001 C CNN
+F 3 "~" H 10650 2800 50  0001 C CNN
+	1    10650 2800
 	1    0    0    -1
 $EndComp
@@
 	1    0    0    -1
 $EndComp
+Wire Wire Line
+	10450 2600 10450 2700
+Wire Wire Line
+	9750 3250 9850 3250
+Wire Wire Line
+	9850 3250 9850 3000
+Wire Wire Line
+	8500 3250 9350 3250
+$Comp
+L Device:C C28
+U 1 1 5FB85B9F
+P 9150 2600
+F 0 "C28" V 9000 2550 50  0000 L CNN
+F 1 "2200" V 9300 2500 50  0000 L CNN
+F 2 "Capacitor_SMD:C_1206_3216Metric" H 9188 2450 50  0001 C CNN
+F 3 "~" H 9150 2600 50  0001 C CNN
+	1    9150 2600
+	0    1    1    0
+$EndComp
+Wire Wire Line
+	8500 2750 8950 2750
+Wire Wire Line
+	8950 2950 8950 2750
+Wire Wire Line
+	9300 2950 9350 2950
+Wire Wire Line
+	9850 3250 10200 3250
+Wire Wire Line
+	10200 3250 10200 2800
+Wire Wire Line
+	10200 2800 10450 2800
+Connection ~ 9850 3250
+Wire Wire Line
+	9850 2700 9850 2600
+Connection ~ 9850 2600
+Wire Wire Line
+	9850 2600 10450 2600
+Wire Wire Line
+	9800 2600 9850 2600
+$Comp
+L power:VPP #PWR058
+U 1 1 5ED3C80C
+P 9800 2600
+F 0 "#PWR058" H 9800 2450 50  0001 C CNN
+F 1 "VPP" V 9800 2800 50  0000 C CNN
+F 2 "" H 9800 2600 50  0001 C CNN
+F 3 "" H 9800 2600 50  0001 C CNN
+	1    9800 2600
+	0    -1   -1   0
+$EndComp
+Wire Wire Line
+	8950 2950 9000 2950
+Wire Wire Line
+	9000 2600 8950 2600
+Wire Wire Line
+	8950 2600 8950 2750
+Connection ~ 8950 2750
+Wire Wire Line
+	9300 2600 9350 2600
+Wire Wire Line
+	9350 2600 9350 2750
+Wire Wire Line
+	9550 2950 9550 2750
+Wire Wire Line
+	9550 2750 9350 2750
+Connection ~ 9350 2750
+Wire Wire Line
+	9350 2750 9350 2950
 $EndSCHEMATC

Commit message: Changed C28 capcity
Parts:
- C28: value 2200 -> 1000
Changed lines of the file:
@@
 P 9150 2600
 F 0 "C28" V 9000 2550 50  0000 L CNN
-F 1 "2200" V 9300 2500 50  0000 L CNN
+F 1 "1000" V 9300 2500 50  0000 L CNN
 F 2 "Capacitor_SMD:C_1206_3216Metric" H 9188 2450 50  0001 C CNN
 F 3 "~" H 9150 2600 50  0001 C CNN

Commit message: Changed footprint of microphone module, added bias voltage to microphone signal, changed power suply of LCD.
Parts:
- added C29: 1.0, Capacitor_SMD:C_1206_3216Metric, symbol Device:C
- added R25, R26: 15K, Resistor_SMD:R_1206_3216Metric, symbol Device:R
Connections:
- net GNDA: now also R26.2
- net VDDA: now also R25.2
- net VPP: no longer C1.1, LCD1.2 (VDD)
- net +5V: now reaches C10.1, C17.1, C3.1, C7.1, J3.1, Q3.2 (S), R10.1, U3.3 (VI)
- net +5V: now also C1.1, LCD1.2 (VDD)
- net at U1.8: now also C29.1, R25.1, R26.1; no longer IC1.4 (OUT)
- new net: C29.2, IC1.4 (OUT)
Changed lines of the file:
@@
-$EndComp
-$Comp
-L power:VPP #PWR048
-U 1 1 5EA4AF3B
-P 7550 2000
-F 0 "#PWR048" H 7550 1850 50  0001 C CNN
-F 1 "VPP" V 7550 2200 50  0000 C CNN
-F 2 "" H 7550 2000 50  0001 C CNN
-F 3 "" H 7550 2000 50  0001 C CNN
-	1    7550 2000
-	-1   0    0    1
 $EndComp
 $Comp
@@
 	650  3800 4150 3800
 Wire Wire Line
-	3000 4100 3850 4100
-Wire Wire Line
 	650  4100 2000 4100
 $Comp
@@
 F 3 "~" H 1150 5550 50  0001 C CNN
 	1    1150 5550
-	1    0    0    -1
-$EndComp
-$Comp
-L power:VPP #PWR01
-U 1 1 5FA6CB83
-P 800 5350
-F 0 "#PWR01" H 800 5200 50  0001 C CNN
-F 1 "VPP" H 800 5500 50  0000 C CNN
-F 2 "" H 800 5350 50  0001 C CNN
-F 3 "" H 800 5350 50  0001 C CNN
-	1    800  5350
 	1    0    0    -1
 $EndComp
@@
 Wire Wire Line
 	9350 2750 9350 2950
+$Comp
+L power:+5V #PWR048
+U 1 1 5FBCF8A2
+P 2050 6400
+F 0 "#PWR048" H 2050 6250 50  0001 C CNN
+F 1 "+5V" H 2065 6573 50  0000 C CNN
+F 2 "" H 2050 6400 50  0001 C CNN
+F 3 "" H 2050 6400 50  0001 C CNN
+	1    2050 6400
+	1    0    0    -1
+$EndComp
+$Comp
+L power:+5V #PWR054
+U 1 1 5FBF906B
+P 7550 2000
+F 0 "#PWR054" H 7550 1850 50  0001 C CNN
+F 1 "+5V" V 7550 2200 50  0000 C CNN
+F 2 "" H 7550 2000 50  0001 C CNN
+F 3 "" H 7550 2000 50  0001 C CNN
+	1    7550 2000
+	-1   0    0    1
+$EndComp
+$Comp
+L power:+5V #PWR01
+U 1 1 5FC0FD2F
+P 800 5350
+F 0 "#PWR01" H 800 5200 50  0001 C CNN
+F 1 "+5V" H 815 5523 50  0000 C CNN
+F 2 "" H 800 5350 50  0001 C CNN
+F 3 "" H 800 5350 50  0001 C CNN
+	1    800  5350
+	1    0    0    -1
+$EndComp
+$Comp
+L Device:R R25
+U 1 1 5FB566D5
+P 3450 4350
+F 0 "R25" H 3600 4400 50  0000 C CNN
+F 1 "15K" H 3600 4300 50  0000 C CNN
+F 2 "Resistor_SMD:R_1206_3216Metric" V 3380 4350 50  0001 C CNN
+F 3 "~" H 3450 4350 50  0001 C CNN
+	1    3450 4350
+	1    0    0    -1
+$EndComp
+$Comp
+L Device:R R26
+U 1 1 5FB57E90
+P 3750 4350
+F 0 "R26" H 3900 4400 50  0000 C CNN
+F 1 "15K" H 3900 4300 50  0000 C CNN
+F 2 "Resistor_SMD:R_1206_3216Metric" V 3680 4350 50  0001 C CNN
+F 3 "~" H 3750 4350 50  0001 C CNN
+	1    3750 4350
+	1    0    0    -1
+$EndComp
+$Comp
+L Device:C C29
+U 1 1 5FB5943C
+P 3150 4100
+F 0 "C29" V 3000 4050 50  0000 L CNN
+F 1 "1.0" V 3300 4050 50  0000 L CNN
+F 2 "Capacitor_SMD:C_1206_3216Metric" H 3188 3950 50  0001 C CNN
+F 3 "~" H 3150 4100 50  0001 C CNN
+	1    3150 4100
+	0    1    1    0
+$EndComp
+Wire Wire Line
+	3300 4100 3450 4100
+Wire Wire Line
+	3450 4100 3450 4200
+Wire Wire Line
+	3450 4100 3750 4100
+Wire Wire Line
+	3750 4100 3750 4200
+Connection ~ 3450 4100
+Wire Wire Line
+	3750 4100 3850 4100
+Connection ~ 3750 4100
+$Comp
+L power:VDDA #PWR062
+U 1 1 5FBBA66F
+P 3450 4550
+F 0 "#PWR062" H 3450 4400 50  0001 C CNN
+F 1 "VDDA" H 3350 4700 50  0000 L CNN
+F 2 "" H 3450 4550 50  0001 C CNN
+F 3 "" H 3450 4550 50  0001 C CNN
+	1    3450 4550
+	-1   0    0    1
+$EndComp
+$Comp
+L power:GNDA #PWR063
+U 1 1 5FBBBE09
+P 3750 4550
+F 0 "#PWR063" H 3750 4300 50  0001 C CNN
+F 1 "GNDA" H 3750 4400 50  0000 C CNN
+F 2 "" H 3750 4550 50  0001 C CNN
+F 3 "" H 3750 4550 50  0001 C CNN
+	1    3750 4550
+	1    0    0    -1
+$EndComp
+Wire Wire Line
+	3450 4500 3450 4550
+Wire Wire Line
+	3750 4500 3750 4550
 $EndSCHEMATC

Commit message: Changed output switch on schematic and pcb
Parts:
- added D3, D4: 1N4148WS, Diode_SMD:D_SOD-323, symbol Diode:1N4148WS
- added R23: 10K, Resistor_SMD:R_1206_3216Metric, symbol Device:R
- renumbered R23 to R27
Connections:
- net IR: now also U4.15 (PD6); no longer U4.14 (PD5)
- net MC_GAIN: now also U4.14 (PD5); no longer U4.15 (PD6)
- net MOSI: now also D3.1 (K); no longer Q4.2 (E)
- net VPP: now also C28.2, R22.2, R23.2
- net WS_LOCK: now also D4.1 (K); no longer C28.2, R22.2
- net at C28.1, Q4.1 (B): now also R23.1; no longer R22.1
- new net: D3.2 (A), D4.2 (A), Q4.2 (E), R22.1
Other:
- moved on the sheet: C28, J6, Q4, R22, R25, R26, R27
